Commit message: resolved the swivel joint
added a fake joint publisher for that continuous joint, in the rviz launchfile.

File: pioneer_3dx_ros/pioneer_description/urdf/pioneer3dx_simple.xacro (robot description, xacro)
@@ -63,5 +63,4 @@
 			<geometry>
 				<mesh filename="package://pioneer_description/meshes/p3dx_meshes/top.stl"/>
-				<!--box size="0.44 0.38 0.005"/-->
 			</geometry>
 		</collision>
@@ -71,7 +70,4 @@
 		<origin xyz="-0.185 0 0.055" rpy="0 0 0"/>
 		<axis xyz="0 0 1"/>
-		<!--<anchor xyz="0 0 0"/>
-  	<limit effort="100" velocity="100" k_velocity="0" />
-  	<joint_properties damping="0.0" friction="0.0" />-->
 		<parent link="base_link"/>
 		<child link="swivel"/>
@@ -99,4 +95,10 @@
 	</link>
 <!-- Center Wheel + Hubcap -->
+	<joint name="swivel_hubcap_joint" type="continuous">
+		<origin xyz="-0.026 0 -0.016" rpy="0 0 0"/>
+		<axis xyz="0 1 0"/>
+	  <parent link="swivel"/>
+		<child link="center_wheel"/>
+	</joint>
 	<link name="center_hubcap">
 		<inertial>
@@ -120,12 +122,8 @@
 	  </collision>
 	</link>
-	<joint name="swivel_hubcap_joint" type="continuous">
-		<origin xyz="-0.026 0 -0.016" rpy="0 0 0"/>
-		<axis xyz="0 1 0"/>
-		<!--<anchor xyz="0 0 0"/>
-    <limit effort="1000" velocity="1000" k_velocity="0" />
-    <joint_properties damping="0.0" friction="0.0" />-->
-	  <parent link="swivel"/>
-		<child link="center_wheel"/>
+	<joint name="center_wheel_joint" type="fixed">
+		<origin xyz="-0.0035 0 -0.001" rpy="0 0 0"/>
+		<parent link="center_wheel"/>
+		<child link="center_hubcap"/>
 	</joint>
 	<link name="center_wheel">
@@ -147,20 +145,11 @@
 		  <geometry>
 		    <mesh filename="package://pioneer_description/meshes/p3dx_meshes/center_wheel.stl"/>
-			  <!--<cylinder radius="0.0375" length="0.03"/>-->
 		  </geometry>
 	  </collision>
 	</link>
-	<joint name="center_wheel_joint" type="fixed">
-		<origin xyz="-0.0035 0 -0.001" rpy="0 0 0"/>
-		<parent link="center_wheel"/>
-		<child link="center_hubcap"/>
-	</joint>
 	<!-- Left Wheel -->
 	<joint name="base_left_wheel_joint" type="continuous">
 		<origin xyz="0 0.155 0.093" rpy="0 0 0"/>
 		<axis xyz="0 1 0"/>
-		<!--<anchor xyz="0 0 0"/>
-  	<limit effort="1000" velocity="1000" k_velocity="0" />
-  	<joint_properties damping="0.0" friction="0.0" />-->
 		<parent link="base_link"/>
 		<child link="left_wheel"/>
