Commit message: laserscan_kinect + some cleanup inside the pioneer_description folder

File: pioneer_3dx_ros/pioneer_description/urdf/pioneer_kinect.urdf.xacro (robot description, xacro)
@@ -5,5 +5,5 @@
 -->
 <robot name="pioneer" xmlns:xacro="http://ros.org/wiki/xacro">
-  <xacro:include filename="$(find pioneer_description)/urdf/pioneer3dx_simple.xacro"/>
+  <xacro:include filename="$(find pioneer_description)/urdf/robot_base/pioneer3dx.xacro"/>
   <xacro:include filename="$(find pioneer_description)/urdf/sensors/kinect.urdf.xacro"/>
   <pioneer3dx/>

File: pioneer_3dx_ros/pioneer_description/urdf/sensors/kinect.urdf.xacro (robot description, xacro)
@@ -1,6 +1,6 @@
 <?xml version="1.0"?>
 <robot name="sensor_kinect" xmlns:xacro="http://ros.org/wiki/xacro">
-  <xacro:include filename="$(find pioneer_description)/urdf/turtlebot_gazebo.urdf.xacro"/>
-  <xacro:include filename="$(find pioneer_description)/urdf/turtlebot_properties.urdf.xacro"/>
+  <xacro:include filename="$(find pioneer_description)/urdf/sensors/kinect_gazebo.urdf.xacro"/>
+  <xacro:include filename="$(find pioneer_description)/urdf/sensors/kinect_properties.urdf.xacro"/>
   <xacro:property name="kinect_cam_py" value="-0.0125"/>
   <!-- Parameterised in part by the values in turtlebot_properties.urdf.xacro -->
@@ -27,5 +27,5 @@
        <origin xyz="0 0 0" rpy="0 0 ${M_PI/2}"/>
         <geometry>
-         <mesh filename="package://turtlebot_description/meshes/sensors/kinect.dae"/>
+         <mesh filename="package://pioneer_description/meshes/sensors/kinect.dae"/>
         </geometry>
       </visual>
@@ -60,5 +60,5 @@
 	<link name="camera_depth_optical_frame"/>
 	<!-- Kinect sensor for simulation -->
-	<turtlebot_sim_3dsensor/>
+	<kinect_sim_3dsensor/>
   </xacro:macro>
 </robot>

File: pioneer_3dx_ros/pioneer_description/urdf/sensors/kinect_gazebo.urdf.xacro (robot description, xacro)
@@ -1,6 +1,6 @@
 <?xml version="1.0"?>
-<robot name="turtlebot_gazebo" xmlns:xacro="http://ros.org/wiki/xacro">
+<robot name="kinect_gazebo" xmlns:xacro="http://ros.org/wiki/xacro">
   <!-- Microsoft Kinect / ASUS Xtion PRO Live for simulation -->
-  <xacro:macro name="turtlebot_sim_3dsensor">
+  <xacro:macro name="kinect_sim_3dsensor">
     <gazebo reference="camera_link">
       <sensor type="depth" name="camera">

File: pioneer_3dx_ros/pioneer_description/urdf/sensors/kinect_properties.urdf.xacro (robot description, xacro)
@@ -19,7 +19,7 @@
      (currently in development and awaiting feedback)
    -->
-	<xacro:property name="cam_px" value="0.107" />
+	<xacro:property name="cam_px" value="0.14" />
 <!--	<xacro:property name="cam_py" value="-0.0125" /> Y varies for different configurations. get sets in sensors_urdf -->
-	<xacro:property name="cam_pz" value="0.2870" />
+	<xacro:property name="cam_pz" value="0.27" />
 	<xacro:property name="cam_or" value="0" />
 	<xacro:property name="cam_op" value="0" />
