Commit message: reconfigure of launchfiles.

File: Resources/pioneer_3dx_ros/pioneer_description/urdf/pioneer_kinect.urdf.xacro (robot description, xacro)
@@ -8,4 +8,4 @@
   <xacro:include filename="$(find pioneer_description)/urdf/sensors/kinect.urdf.xacro"/>
   <pioneer3dx/>
-  <sensor_kinect parent="base_link"/>
+  <sensor_kinect parent="top"/>
 </robot>

File: Resources/pioneer_3dx_ros/pioneer_description/urdf/pioneer_kinect_real.urdf.xacro (robot description, xacro)
@@ -8,4 +8,4 @@
   <xacro:include filename="$(find pioneer_description)/urdf/sensors/kinect_real.urdf.xacro"/>
   <pioneer3dx/>
-  <sensor_kinect parent="base_link"/>
+  <sensor_kinect parent="top"/>
 </robot>

File: Resources/pioneer_3dx_ros/pioneer_description/urdf/sensors/kinect_properties.urdf.xacro (robot description, xacro)
@@ -21,5 +21,5 @@
 	<xacro:property name="cam_px" value="0.14" />
 <!--	<xacro:property name="cam_py" value="-0.0125" /> Y varies for different configurations. get sets in sensors_urdf -->
-	<xacro:property name="cam_pz" value="0.27" />
+	<xacro:property name="cam_pz" value="0.05" />
 	<xacro:property name="cam_or" value="0" />
 	<xacro:property name="cam_op" value="0" />
